File: POV_display_schematic/POV_display_schematic.kicad_pcb (KiCad board)
At the start: 2 copper layers, 200 x 20 mm, 124 parts, among them J1 Conn_01x05_Female, J2 Conn_01x02_Male, Q1 MMBT3904, Q2 MMBT3906, U1 74HC595, U10 74HC595, U11 HT75xx-1-SOT89, U2 74HC595, U3 74HC595, U4 74HC595, U5 74HC595, U6 LN4913, U7 74HC595, U8 74HC595, U9 STM32L051C8Tx, Y1 32.768 KHz

Commit message: Uploaded offline work
Parts:
- removed the C11 at (210.9, 105.1)
- removed the C13 at (221.9, 97.3)
- removed the C14 at (68.2, 98.5)
- removed the C6 at (232.2, 96.4)
- removed the C9 at (211.2, 90.4)
- removed J2: Conn_01x02_Male, Connector_PinHeader_2.54mm:PinHeader_1x02_P2.54mm_Vertical
- removed Q1: MMBT3904, Package_TO_SOT_SMD:TSOT-23_HandSoldering
- removed the R64 at (220.4, 101.5)
- removed the R65 at (228.6, 92.9)
- removed the R66 at (224.2, 103.7)
- removed the R67 at (240.1, 103.7)
- removed the R68 at (240.1, 101.1)
- removed the R69 at (217.5, 89.6)
- removed the U11 at (233.2, 94.6)
- removed the U3 at (155.3, 97.2)
- removed the U6 at (225.6, 101.5)
- added C1: 10uF, Capacitor_SMD:C_0805_2012Metric_Pad1.18x1.45mm_HandSolder, F.Cu at (212.8, 83.3)
- added C10: 100nF, Capacitor_SMD:C_0805_2012Metric_Pad1.18x1.45mm_HandSolder, F.Cu at (227.7, 103.2)
- added C18: 10pF, Capacitor_SMD:C_0603_1608Metric_Pad1.08x0.95mm_HandSolder, F.Cu at (240.8, 96.8)
- added C2: 10uF, Capacitor_SMD:C_0805_2012Metric_Pad1.18x1.45mm_HandSolder, F.Cu at (232.5, 88.9)
- added C3: 10uF, Capacitor_SMD:C_0805_2012Metric_Pad1.18x1.45mm_HandSolder, F.Cu at (212.7, 87.0)
- added C4: 10uF, Capacitor_SMD:C_0805_2012Metric_Pad1.18x1.45mm_HandSolder, F.Cu at (224.3, 84.4)
- added D1: Green, LED_SMD:LED_0805_2012Metric_Pad1.15x1.40mm_HandSolder, F.Cu at (240.8, 84.8)
- added D2: Red, LED_SMD:LED_0805_2012Metric_Pad1.15x1.40mm_HandSolder, F.Cu at (240.8, 82.0)
- added D24: D_Photo, LED_THT:LED_D5.0mm, B.Cu at (264.8, 97.5)
- added H1: M3, MountingHole:MountingHole_3.2mm_M3, F.Cu at (213.8, 118.2)
- added H2: M3, MountingHole:MountingHole_3.2mm_M3, F.Cu at (256.2, 76.8)
- added H3: M3, MountingHole:MountingHole_3.2mm_M3, F.Cu at (256.2, 118.2)
- added H4: M3, MountingHole:MountingHole_3.2mm_M3, F.Cu at (213.8, 76.8)
- added J3: HC05/06 Port, Connector_PinHeader_2.54mm:PinHeader_1x04_P2.54mm_Vertical, F.Cu at (231.0, 76.8)
- added J4: 6PinDebugPort, Connector_IDC:IDC-Header_2x03_P2.54mm_Vertical, F.Cu at (266.5, 86.8)
- added Q3: MMBT3906, Package_TO_SOT_SMD:TSOT-23_HandSoldering, F.Cu at (246.9, 81.2)
- added R1: 1K, Resistor_SMD:R_0805_2012Metric_Pad1.20x1.40mm_HandSolder, F.Cu at (236.3, 84.9)
- added R10: 10K, Resistor_SMD:R_0805_2012Metric_Pad1.20x1.40mm_HandSolder, F.Cu at (218.9, 110.2)
- added R11: 10K, Resistor_SMD:R_0805_2012Metric_Pad1.20x1.40mm_HandSolder, F.Cu at (246.6, 110.2)
- added R2: 1K, Resistor_SMD:R_0805_2012Metric_Pad1.20x1.40mm_HandSolder, F.Cu at (236.3, 82.0)
- added R3: 47K, Resistor_SMD:R_0805_2012Metric_Pad1.20x1.40mm_HandSolder, F.Cu at (263.1, 109.0)
- added R4: 47K, Resistor_SMD:R_0805_2012Metric_Pad1.20x1.40mm_HandSolder, F.Cu at (263.1, 111.9)
- added R5: 4K7, Resistor_SMD:R_0805_2012Metric_Pad1.20x1.40mm_HandSolder, F.Cu at (224.8, 89.0)
- added R6: 47K, Resistor_SMD:R_0805_2012Metric_Pad1.20x1.40mm_HandSolder, F.Cu at (249.9, 87.2)
- added R7: 10K, Resistor_SMD:R_0805_2012Metric_Pad1.20x1.40mm_HandSolder, F.Cu at (259.6, 97.5)
- added R8: 47K, Resistor_SMD:R_0805_2012Metric_Pad1.20x1.40mm_HandSolder, F.Cu at (246.9, 87.2)
- added R9: 10K, Resistor_SMD:R_0805_2012Metric_Pad1.20x1.40mm_HandSolder, F.Cu at (244.2, 87.2)
- added SW1: RST, custom_buttons_switches:TSB008, F.Cu at (223.5, 112.0)
- added SW2: BOOT, custom_buttons_switches:TSB008, F.Cu at (236.0, 112.0)
- added TP1: TestPoint, TestPoint:TestPoint_Pad_2.0x2.0mm, F.Cu at (226.0, 118.2)
- added TP2: TestPoint, TestPoint:TestPoint_Pad_2.0x2.0mm, F.Cu at (221.0, 118.2)
- added TP3: TestPoint, TestPoint:TestPoint_Pad_2.0x2.0mm, F.Cu at (241.0, 118.2)
- added TP4: TestPoint, TestPoint:TestPoint_Pad_2.0x2.0mm, F.Cu at (236.0, 118.2)
- added TP5: TestPoint, TestPoint:TestPoint_Pad_2.0x2.0mm, F.Cu at (246.0, 118.2)
- added TP6: TestPoint, TestPoint:TestPoint_Pad_2.0x2.0mm, F.Cu at (231.0, 118.2)
- added U1: HT7325, Package_TO_SOT_SMD:SOT-89-3_Handsoldering, F.Cu at (219.3, 83.3)
- added U2: TP4056, Package_SO:SOP-8_3.9x4.9mm_P1.27mm, F.Cu at (229.6, 83.6)
- added U7: 74HC595, Package_SO:SO-16_3.9x9.9mm_P1.27mm, B.Cu at (155.3, 97.2)
- BT1: value Battery_Cell -> LiPo battery
- C11: renamed from C5; footprint Capacitor_SMD:C_1206_3216Metric_Pad1.33x1.80mm_HandSolder -> Capacitor_SMD:C_0805_2012Metric_Pad1.18x1.45mm_HandSolder
- C12: value 10pF -> 100nF; footprint Capacitor_SMD:C_0603_1608Metric_Pad1.08x0.95mm_HandSolder -> Capacitor_SMD:C_0805_2012Metric_Pad1.18x1.45mm_HandSolder
- C13: renamed from C7; footprint Capacitor_SMD:C_1206_3216Metric_Pad1.33x1.80mm_HandSolder -> Capacitor_SMD:C_0805_2012Metric_Pad1.18x1.45mm_HandSolder
- C14: renamed from C10; footprint Capacitor_SMD:C_1206_3216Metric_Pad1.33x1.80mm_HandSolder -> Capacitor_SMD:C_0805_2012Metric_Pad1.18x1.45mm_HandSolder
- C15: value 10uF -> 100nF; footprint Capacitor_SMD:C_1206_3216Metric_Pad1.33x1.80mm_HandSolder -> Capacitor_SMD:C_0805_2012Metric_Pad1.18x1.45mm_HandSolder; moved to F.Cu
- C16: value 10uF -> 1uF; footprint Capacitor_SMD:C_1206_3216Metric_Pad1.33x1.80mm_HandSolder -> Capacitor_SMD:C_0805_2012Metric_Pad1.18x1.45mm_HandSolder
- C17: value 100nF -> 10pF; footprint Capacitor_SMD:C_1206_3216Metric_Pad1.33x1.80mm_HandSolder -> Capacitor_SMD:C_0603_1608Metric_Pad1.08x0.95mm_HandSolder; moved to F.Cu
- C5: renamed from C1; footprint Capacitor_SMD:C_1206_3216Metric_Pad1.33x1.80mm_HandSolder -> Capacitor_SMD:C_0805_2012Metric_Pad1.18x1.45mm_HandSolder
- C6: renamed from C2; footprint Capacitor_SMD:C_1206_3216Metric_Pad1.33x1.80mm_HandSolder -> Capacitor_SMD:C_0805_2012Metric_Pad1.18x1.45mm_HandSolder
- C7: renamed from C3; footprint Capacitor_SMD:C_1206_3216Metric_Pad1.33x1.80mm_HandSolder -> Capacitor_SMD:C_0805_2012Metric_Pad1.18x1.45mm_HandSolder
- C8: footprint Capacitor_SMD:C_1206_3216Metric_Pad1.33x1.80mm_HandSolder -> Capacitor_SMD:C_0805_2012Metric_Pad1.18x1.45mm_HandSolder
- C9: renamed from C4; footprint Capacitor_SMD:C_1206_3216Metric_Pad1.33x1.80mm_HandSolder -> Capacitor_SMD:C_0805_2012Metric_Pad1.18x1.45mm_HandSolder
- J1: value Conn_01x05_Female -> USB_B_Micro; footprint Connector_PinHeader_2.54mm:PinHeader_1x05_P2.54mm_Vertical -> Connector_USB:USB_Micro-B_Molex-105017-0001
- Q2: value MMBT3906 -> MMBT3904; moved to F.Cu
- R12: renamed from R1; footprint Resistor_SMD:R_0603_1608Metric_Pad0.98x0.95mm_HandSolder -> Resistor_SMD:R_0603_1608Metric
- R13: renamed from R2; footprint Resistor_SMD:R_0603_1608Metric_Pad0.98x0.95mm_HandSolder -> Resistor_SMD:R_0603_1608Metric
- R14: renamed from R3; footprint Resistor_SMD:R_0603_1608Metric_Pad0.98x0.95mm_HandSolder -> Resistor_SMD:R_0603_1608Metric
- R15: renamed from R4; footprint Resistor_SMD:R_0603_1608Metric_Pad0.98x0.95mm_HandSolder -> Resistor_SMD:R_0603_1608Metric
- R16: renamed from R5; footprint Resistor_SMD:R_0603_1608Metric_Pad0.98x0.95mm_HandSolder -> Resistor_SMD:R_0603_1608Metric
- R17: renamed from R6; footprint Resistor_SMD:R_0603_1608Metric_Pad0.98x0.95mm_HandSolder -> Resistor_SMD:R_0603_1608Metric
- R18: renamed from R7; footprint Resistor_SMD:R_0603_1608Metric_Pad0.98x0.95mm_HandSolder -> Resistor_SMD:R_0603_1608Metric
- R19: renamed from R8; footprint Resistor_SMD:R_0603_1608Metric_Pad0.98x0.95mm_HandSolder -> Resistor_SMD:R_0603_1608Metric
- R20: renamed from R9; footprint Resistor_SMD:R_0603_1608Metric_Pad0.98x0.95mm_HandSolder -> Resistor_SMD:R_0603_1608Metric
- R21: renamed from R10; footprint Resistor_SMD:R_0603_1608Metric_Pad0.98x0.95mm_HandSolder -> Resistor_SMD:R_0603_1608Metric
- R22: renamed from R11; footprint Resistor_SMD:R_0603_1608Metric_Pad0.98x0.95mm_HandSolder -> Resistor_SMD:R_0603_1608Metric
- R23: renamed from R12; footprint Resistor_SMD:R_0603_1608Metric_Pad0.98x0.95mm_HandSolder -> Resistor_SMD:R_0603_1608Metric
- R24: renamed from R13; footprint Resistor_SMD:R_0603_1608Metric_Pad0.98x0.95mm_HandSolder -> Resistor_SMD:R_0603_1608Metric
- R25: renamed from R14; footprint Resistor_SMD:R_0603_1608Metric_Pad0.98x0.95mm_HandSolder -> Resistor_SMD:R_0603_1608Metric
- R26: renamed from R15; footprint Resistor_SMD:R_0603_1608Metric_Pad0.98x0.95mm_HandSolder -> Resistor_SMD:R_0603_1608Metric
- R27: renamed from R16; footprint Resistor_SMD:R_0603_1608Metric_Pad0.98x0.95mm_HandSolder -> Resistor_SMD:R_0603_1608Metric
- R28: renamed from R17; footprint Resistor_SMD:R_0603_1608Metric_Pad0.98x0.95mm_HandSolder -> Resistor_SMD:R_0603_1608Metric
- R29: renamed from R18; footprint Resistor_SMD:R_0603_1608Metric_Pad0.98x0.95mm_HandSolder -> Resistor_SMD:R_0603_1608Metric
- R30: renamed from R19; footprint Resistor_SMD:R_0603_1608Metric_Pad0.98x0.95mm_HandSolder -> Resistor_SMD:R_0603_1608Metric
- R31: renamed from R20; footprint Resistor_SMD:R_0603_1608Metric_Pad0.98x0.95mm_HandSolder -> Resistor_SMD:R_0603_1608Metric
- R32: renamed from R21; footprint Resistor_SMD:R_0603_1608Metric_Pad0.98x0.95mm_HandSolder -> Resistor_SMD:R_0603_1608Metric
- R33: renamed from R22; footprint Resistor_SMD:R_0603_1608Metric_Pad0.98x0.95mm_HandSolder -> Resistor_SMD:R_0603_1608Metric
- R34: renamed from R23; footprint Resistor_SMD:R_0603_1608Metric_Pad0.98x0.95mm_HandSolder -> Resistor_SMD:R_0603_1608Metric
- R35: renamed from R24; footprint Resistor_SMD:R_0603_1608Metric_Pad0.98x0.95mm_HandSolder -> Resistor_SMD:R_0603_1608Metric
- R36: renamed from R25; footprint Resistor_SMD:R_0603_1608Metric_Pad0.98x0.95mm_HandSolder -> Resistor_SMD:R_0603_1608Metric
- R37: renamed from R26; footprint Resistor_SMD:R_0603_1608Metric_Pad0.98x0.95mm_HandSolder -> Resistor_SMD:R_0603_1608Metric
- R38: renamed from R27; footprint Resistor_SMD:R_0603_1608Metric_Pad0.98x0.95mm_HandSolder -> Resistor_SMD:R_0603_1608Metric
- R39: renamed from R28; footprint Resistor_SMD:R_0603_1608Metric_Pad0.98x0.95mm_HandSolder -> Resistor_SMD:R_0603_1608Metric
- R40: renamed from R29; footprint Resistor_SMD:R_0603_1608Metric_Pad0.98x0.95mm_HandSolder -> Resistor_SMD:R_0603_1608Metric
- R41: renamed from R30; footprint Resistor_SMD:R_0603_1608Metric_Pad0.98x0.95mm_HandSolder -> Resistor_SMD:R_0603_1608Metric
- R42: renamed from R31; footprint Resistor_SMD:R_0603_1608Metric_Pad0.98x0.95mm_HandSolder -> Resistor_SMD:R_0603_1608Metric
- R43: renamed from R32; footprint Resistor_SMD:R_0603_1608Metric_Pad0.98x0.95mm_HandSolder -> Resistor_SMD:R_0603_1608Metric
- R44: renamed from R33; footprint Resistor_SMD:R_0603_1608Metric_Pad0.98x0.95mm_HandSolder -> Resistor_SMD:R_0603_1608Metric
- R45: renamed from R34; footprint Resistor_SMD:R_0603_1608Metric_Pad0.98x0.95mm_HandSolder -> Resistor_SMD:R_0603_1608Metric
- R46: renamed from R35; footprint Resistor_SMD:R_0603_1608Metric_Pad0.98x0.95mm_HandSolder -> Resistor_SMD:R_0603_1608Metric
- R47: renamed from R36; footprint Resistor_SMD:R_0603_1608Metric_Pad0.98x0.95mm_HandSolder -> Resistor_SMD:R_0603_1608Metric
- R48: renamed from R37; footprint Resistor_SMD:R_0603_1608Metric_Pad0.98x0.95mm_HandSolder -> Resistor_SMD:R_0603_1608Metric
- R49: renamed from R38; footprint Resistor_SMD:R_0603_1608Metric_Pad0.98x0.95mm_HandSolder -> Resistor_SMD:R_0603_1608Metric
- R50: renamed from R39; footprint Resistor_SMD:R_0603_1608Metric_Pad0.98x0.95mm_HandSolder -> Resistor_SMD:R_0603_1608Metric
- R51: renamed from R40; footprint Resistor_SMD:R_0603_1608Metric_Pad0.98x0.95mm_HandSolder -> Resistor_SMD:R_0603_1608Metric
- R52: renamed from R41; footprint Resistor_SMD:R_0603_1608Metric_Pad0.98x0.95mm_HandSolder -> Resistor_SMD:R_0603_1608Metric
- R53: renamed from R42; footprint Resistor_SMD:R_0603_1608Metric_Pad0.98x0.95mm_HandSolder -> Resistor_SMD:R_0603_1608Metric
- R54: renamed from R43; footprint Resistor_SMD:R_0603_1608Metric_Pad0.98x0.95mm_HandSolder -> Resistor_SMD:R_0603_1608Metric
- R55: renamed from R44; footprint Resistor_SMD:R_0603_1608Metric_Pad0.98x0.95mm_HandSolder -> Resistor_SMD:R_0603_1608Metric
- R56: renamed from R45; footprint Resistor_SMD:R_0603_1608Metric_Pad0.98x0.95mm_HandSolder -> Resistor_SMD:R_0603_1608Metric
- R57: renamed from R46; footprint Resistor_SMD:R_0603_1608Metric_Pad0.98x0.95mm_HandSolder -> Resistor_SMD:R_0603_1608Metric
- R58: renamed from R47; footprint Resistor_SMD:R_0603_1608Metric_Pad0.98x0.95mm_HandSolder -> Resistor_SMD:R_0603_1608Metric
- R59: renamed from R48; footprint Resistor_SMD:R_0603_1608Metric_Pad0.98x0.95mm_HandSolder -> Resistor_SMD:R_0603_1608Metric
- R60: renamed from R49; footprint Resistor_SMD:R_0603_1608Metric_Pad0.98x0.95mm_HandSolder -> Resistor_SMD:R_0603_1608Metric
- R61: renamed from R50; footprint Resistor_SMD:R_0603_1608Metric_Pad0.98x0.95mm_HandSolder -> Resistor_SMD:R_0603_1608Metric
- R62: renamed from R51; footprint Resistor_SMD:R_0603_1608Metric_Pad0.98x0.95mm_HandSolder -> Resistor_SMD:R_0603_1608Metric
- R63: renamed from R52; footprint Resistor_SMD:R_0603_1608Metric_Pad0.98x0.95mm_HandSolder -> Resistor_SMD:R_0603_1608Metric
- R64: renamed from R53; footprint Resistor_SMD:R_0603_1608Metric_Pad0.98x0.95mm_HandSolder -> Resistor_SMD:R_0603_1608Metric
- R65: renamed from R54; footprint Resistor_SMD:R_0603_1608Metric_Pad0.98x0.95mm_HandSolder -> Resistor_SMD:R_0603_1608Metric
- R66: renamed from R55; footprint Resistor_SMD:R_0603_1608Metric_Pad0.98x0.95mm_HandSolder -> Resistor_SMD:R_0603_1608Metric
- R67: renamed from R56; footprint Resistor_SMD:R_0603_1608Metric_Pad0.98x0.95mm_HandSolder -> Resistor_SMD:R_0603_1608Metric
- R68: renamed from R57; footprint Resistor_SMD:R_0603_1608Metric_Pad0.98x0.95mm_HandSolder -> Resistor_SMD:R_0603_1608Metric
- R69: renamed from R58; footprint Resistor_SMD:R_0603_1608Metric_Pad0.98x0.95mm_HandSolder -> Resistor_SMD:R_0603_1608Metric
- R70: renamed from R59; footprint Resistor_SMD:R_0603_1608Metric_Pad0.98x0.95mm_HandSolder -> Resistor_SMD:R_0603_1608Metric
- R71: renamed from R60; footprint Resistor_SMD:R_0603_1608Metric_Pad0.98x0.95mm_HandSolder -> Resistor_SMD:R_0603_1608Metric
- R72: renamed from R61; footprint Resistor_SMD:R_0603_1608Metric_Pad0.98x0.95mm_HandSolder -> Resistor_SMD:R_0603_1608Metric
- R73: renamed from R62; footprint Resistor_SMD:R_0603_1608Metric_Pad0.98x0.95mm_HandSolder -> Resistor_SMD:R_0603_1608Metric
- R74: renamed from R63; footprint Resistor_SMD:R_0603_1608Metric_Pad0.98x0.95mm_HandSolder -> Resistor_SMD:R_0603_1608Metric
- moved C16 159.7 mm to (68.2, 97.5), turned to 90 degrees
- moved C8 35.1 mm to (240.0, 103.2), turned to 0 degrees
- moved C17 27.2 mm to (240.8, 100.4), turned to 90 degrees
- moved J1 26.6 mm to (269.8, 107.8), turned to 90 degrees
- moved Q2 26.1 mm to (250.9, 81.2), turned to 90 degrees
- moved BT1 25.2 mm to (221.9, 76.7), turned to 270 degrees
- moved U9 20.9 mm to (234.0, 98.0)
- moved Y1 20.2 mm to (243.0, 99.7), turned to 270 degrees
- moved C15 5.29 mm to (241.4, 92.5)
- moved C12 4.77 mm to (227.5, 92.8)
- moved C9 1.45 mm to (126.0, 97.5)
- moved C11 1.05 mm to (107.0, 97.5)
- moved C14 1.04 mm to (52.0, 97.5)
- moved C13 1.00 mm to (88.0, 97.5)
- moved C6 0.95 mm to (162.8, 97.5)
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- renumbered D8 to D10, D9 to D11, D10 to D12, D11 to D13, D12 to D14, D13 to D15, D14 to D16, D15 to D17, D16 to D18, D17 to D19, D18 to D20, D19 to D21, D20 to D22, D21 to D23, D1 to D3, D2 to D4, D3 to D5, D4 to D6, D5 to D7, D6 to D8, D7 to D9, U4 to U10, U10 to U11, U5 to U3, U1 to U4, U2 to U5, U7 to U6
Connections:
- C12 pad 1: GND -> VCC
- C12 pad 2: Net-(C12-Pad2) -> GND
- C15 pad 1: +BATT -> VCC
- C17 pad 1: VCC -> GND
- C17 pad 2: GND -> Net-(C17-Pad2)
- J1 pad 1: VCC -> +5V
- J1 pad 2: /~rst -> (no net)
- J1 pad 3: /SWDIO -> (no net)
- J1 pad 4: /SWCLK -> GND
- Q2 pad 2: +BATT -> GND
- U10 pad 9: Net-(U4-Pad9) (its old number) -> /SIPO_OUT_4
- U3 pad 14: Net-(U4-Pad9) (its old number) -> /SIPO_OUT_4
- U9 pad 10: /BAT_IN -> (no net)
- U9 pad 12: (no net) -> /BAT_EN
- U9 pad 13: (no net) -> /BAT_IN
- U9 pad 2: (no net) -> /FDBK
- U9 pad 3: Net-(C12-Pad2) -> Net-(C17-Pad2)
- U9 pad 30: (no net) -> /MCU_TX
- U9 pad 31: (no net) -> /MCU_RX
- U9 pad 41: /hall_sig -> (no net)
- U9 pad 46: /BAT_EN -> /USB_Flag
- Y1 pad 2: Net-(C12-Pad2) -> Net-(C17-Pad2)
Routing:
- net VCC: track 314.4 -> 427.4 mm, vias 12 -> 10
- net +5V: track 0.00 -> 98.4 mm, vias 0 -> 2
- net +BATT: track 21.8 -> 82.6 mm, vias 0 -> 4
- net /FDBK: track 0.00 -> 46.6 mm, vias 0 -> 3
- net Net-(U4-Pad9) (its old number): track 32.8 -> 0.00 mm, vias 2 -> 0
- net /SIPO_OUT_4: track 0.00 -> 32.8 mm, vias 0 -> 2
- net /USB_Flag: track 0.00 -> 32.5 mm, vias 0 -> 2
- net /MCU_TX: track 0.00 -> 27.1 mm, vias 0 -> 1
- net /MCU_RX: track 0.00 -> 25.6 mm, vias 0 -> 1
- net /SPI_CLK: track 163.6 -> 185.3 mm
- net /~CLEAR: track 181.5 -> 202.6 mm
- net /SPI_MOSI: track 31.2 -> 52.2 mm
- net /RCLK: track 169.2 -> 190.1 mm
- net /~OE: track 179.6 -> 200.1 mm
- net /~rst: track 42.3 -> 60.1 mm, vias 0 -> 2
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Other:
- board size 200 x 20 mm -> 222.5 x 49 mm
- board text added: "+ -"
- board text added: "+5V"
- board text added: "+Bat"
- board text added: "- +"
- board text added: "ADC in"
- board text added: "FDBK"
- board text added: "Li-Pol Akyga 980 mAh 1S 3,7 V"
- board text added: "Persistance Of Vision by Maciej Krysztowiak"
- board text added: "V02"
- board text added: "VCC/---- ~RST~/SWDIO SWCLK/GND"
- board text added: "Vcc / Gnd / TX / RX"
- board text removed: "+"
- board text removed: "-"
- board text removed: "Flash"
- board text removed: "POV CLOCK by MKrysz"
- board text removed: "SWCLK"
- board text removed: "SWDIO"
- board text removed: "V01"
- board text removed: "~RST"

Commit message: LEDs footprints are now in correct orientation
Parts:
- D10, D11, D12, D13, D14, D15, D16, D17, D18, D19, D20, D21, D22, D23, D3, D4, D5, D6, D7, D8, D9: value LED_RGB -> POV_LED
- turned D8 to 270 degrees
- turned D10 to 270 degrees
- turned D11 to 270 degrees
- turned D12 to 270 degrees
- turned D13 to 270 degrees
- turned D14 to 270 degrees
- turned D15 to 270 degrees
- turned D16 to 270 degrees
- turned D17 to 270 degrees
- turned D18 to 270 degrees
- turned D19 to 270 degrees
- turned D20 to 270 degrees
- turned D21 to 270 degrees
- turned D22 to 270 degrees
- turned D23 to 270 degrees
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Connections:
- D10 pad 1: GND -> Net-(D10-Pad1)
- D10 pad 2: GND -> Net-(D10-Pad2)
- D10 pad 3: GND -> Net-(D10-Pad3)
- D10 pad 4: Net-(D10-Pad4) -> GND
- D10 pad 5: Net-(D10-Pad5) -> GND
- D10 pad 6: Net-(D10-Pad6) -> GND
- D11 pad 1: GND -> Net-(D11-Pad1)
- D11 pad 2: GND -> Net-(D11-Pad2)
- D11 pad 3: GND -> Net-(D11-Pad3)
- D11 pad 4: Net-(D11-Pad4) -> GND
- D11 pad 5: Net-(D11-Pad5) -> GND
- D11 pad 6: Net-(D11-Pad6) -> GND
- D12 pad 1: GND -> Net-(D12-Pad1)
- D12 pad 2: GND -> Net-(D12-Pad2)
- D12 pad 3: GND -> Net-(D12-Pad3)
- D12 pad 4: Net-(D12-Pad4) -> GND
- D12 pad 5: Net-(D12-Pad5) -> GND
- D12 pad 6: Net-(D12-Pad6) -> GND
- D13 pad 1: GND -> Net-(D13-Pad1)
- D13 pad 2: GND -> Net-(D13-Pad2)
- D13 pad 3: GND -> Net-(D13-Pad3)
- D13 pad 4: Net-(D13-Pad4) -> GND
- D13 pad 5: Net-(D13-Pad5) -> GND
- D13 pad 6: Net-(D13-Pad6) -> GND
- D14 pad 1: GND -> Net-(D14-Pad1)
- D14 pad 2: GND -> Net-(D14-Pad2)
- D14 pad 3: GND -> Net-(D14-Pad3)
- D14 pad 4: Net-(D14-Pad4) -> GND
- D14 pad 5: Net-(D14-Pad5) -> GND
- D14 pad 6: Net-(D14-Pad6) -> GND
- D15 pad 1: GND -> Net-(D15-Pad1)
- D15 pad 2: GND -> Net-(D15-Pad2)
- D15 pad 3: GND -> Net-(D15-Pad3)
- D15 pad 4: Net-(D15-Pad4) -> GND
- D15 pad 5: Net-(D15-Pad5) -> GND
- D15 pad 6: Net-(D15-Pad6) -> GND
- D16 pad 1: GND -> Net-(D16-Pad1)
- D16 pad 2: GND -> Net-(D16-Pad2)
- D16 pad 3: GND -> Net-(D16-Pad3)
- D16 pad 4: Net-(D16-Pad4) -> GND
- D16 pad 5: Net-(D16-Pad5) -> GND
- D16 pad 6: Net-(D16-Pad6) -> GND
- D17 pad 1: GND -> Net-(D17-Pad1)
- D17 pad 2: GND -> Net-(D17-Pad2)
- D17 pad 3: GND -> Net-(D17-Pad3)
- D17 pad 4: Net-(D17-Pad4) -> GND
- D17 pad 5: Net-(D17-Pad5) -> GND
- D17 pad 6: Net-(D17-Pad6) -> GND
- D18 pad 1: GND -> Net-(D18-Pad1)
- D18 pad 2: GND -> Net-(D18-Pad2)
- D18 pad 3: GND -> Net-(D18-Pad3)
- D18 pad 4: Net-(D18-Pad4) -> GND
- D18 pad 5: Net-(D18-Pad5) -> GND
- D18 pad 6: Net-(D18-Pad6) -> GND
- D19 pad 1: GND -> Net-(D19-Pad1)
- D19 pad 2: GND -> Net-(D19-Pad2)
- D19 pad 3: GND -> Net-(D19-Pad3)
- D19 pad 4: Net-(D19-Pad4) -> GND
- D19 pad 5: Net-(D19-Pad5) -> GND
- D19 pad 6: Net-(D19-Pad6) -> GND
- D20 pad 1: GND -> Net-(D20-Pad1)
- D20 pad 2: GND -> Net-(D20-Pad2)
- D20 pad 3: GND -> Net-(D20-Pad3)
- D20 pad 4: Net-(D20-Pad4) -> GND
- D20 pad 5: Net-(D20-Pad5) -> GND
- D20 pad 6: Net-(D20-Pad6) -> GND
- D21 pad 1: GND -> Net-(D21-Pad1)
- D21 pad 2: GND -> Net-(D21-Pad2)
- D21 pad 3: GND -> Net-(D21-Pad3)
- D21 pad 4: Net-(D21-Pad4) -> GND
- D21 pad 5: Net-(D21-Pad5) -> GND
- D21 pad 6: Net-(D21-Pad6) -> GND
- D22 pad 1: GND -> Net-(D22-Pad1)
- D22 pad 2: GND -> Net-(D22-Pad2)
- D22 pad 3: GND -> Net-(D22-Pad3)
- D22 pad 4: Net-(D22-Pad4) -> GND
- D22 pad 5: Net-(D22-Pad5) -> GND
- D22 pad 6: Net-(D22-Pad6) -> GND
- D23 pad 1: GND -> Net-(D23-Pad1)
- D23 pad 2: GND -> Net-(D23-Pad2)
- D23 pad 3: GND -> Net-(D23-Pad3)
- D23 pad 4: Net-(D23-Pad4) -> GND
- D23 pad 5: Net-(D23-Pad5) -> GND
- D23 pad 6: Net-(D23-Pad6) -> GND
- D3 pad 1: GND -> Net-(D3-Pad1)
- D3 pad 2: GND -> Net-(D3-Pad2)
- D3 pad 3: GND -> Net-(D3-Pad3)
- D3 pad 4: Net-(D3-Pad4) -> GND
- D3 pad 5: Net-(D3-Pad5) -> GND
- D3 pad 6: Net-(D3-Pad6) -> GND
- D4 pad 1: GND -> Net-(D4-Pad1)
- D4 pad 2: GND -> Net-(D4-Pad2)
- D4 pad 3: GND -> Net-(D4-Pad3)
- D4 pad 4: Net-(D4-Pad4) -> GND
- D4 pad 5: Net-(D4-Pad5) -> GND
- D4 pad 6: Net-(D4-Pad6) -> GND
- D5 pad 1: GND -> Net-(D5-Pad1)
- D5 pad 2: GND -> Net-(D5-Pad2)
- D5 pad 3: GND -> Net-(D5-Pad3)
- D5 pad 4: Net-(D5-Pad4) -> GND
- D5 pad 5: Net-(D5-Pad5) -> GND
- D5 pad 6: Net-(D5-Pad6) -> GND
- D6 pad 1: GND -> Net-(D6-Pad1)
- D6 pad 2: GND -> Net-(D6-Pad2)
- D6 pad 3: GND -> Net-(D6-Pad3)
- D6 pad 4: Net-(D6-Pad4) -> GND
- D6 pad 5: Net-(D6-Pad5) -> GND
- D6 pad 6: Net-(D6-Pad6) -> GND
- D7 pad 1: GND -> Net-(D7-Pad1)
- D7 pad 2: GND -> Net-(D7-Pad2)
- D7 pad 3: GND -> Net-(D7-Pad3)
- D7 pad 4: Net-(D7-Pad4) -> GND
- D7 pad 5: Net-(D7-Pad5) -> GND
- D7 pad 6: Net-(D7-Pad6) -> GND
- D8 pad 1: GND -> Net-(D8-Pad1)
- D8 pad 2: GND -> Net-(D8-Pad2)
- D8 pad 3: GND -> Net-(D8-Pad3)
- D8 pad 4: Net-(D8-Pad4) -> GND
- D8 pad 5: Net-(D8-Pad5) -> GND
- D8 pad 6: Net-(D8-Pad6) -> GND
- D9 pad 1: GND -> Net-(D9-Pad1)
- D9 pad 2: GND -> Net-(D9-Pad2)
- D9 pad 3: GND -> Net-(D9-Pad3)
- D9 pad 4: Net-(D9-Pad4) -> GND
- D9 pad 5: Net-(D9-Pad5) -> GND
- D9 pad 6: Net-(D9-Pad6) -> GND
- R12 pad 2: Net-(D3-Pad6) -> Net-(D3-Pad3)
- R13 pad 2: Net-(D4-Pad6) -> Net-(D4-Pad3)
- R14 pad 2: Net-(D5-Pad6) -> Net-(D5-Pad3)
- R15 pad 2: Net-(D6-Pad6) -> Net-(D6-Pad3)
- R16 pad 2: Net-(D7-Pad6) -> Net-(D7-Pad3)
- R17 pad 2: Net-(D8-Pad6) -> Net-(D8-Pad3)
- R18 pad 2: Net-(D9-Pad6) -> Net-(D9-Pad3)
- R19 pad 2: Net-(D3-Pad5) -> Net-(D3-Pad2)
- R20 pad 2: Net-(D4-Pad5) -> Net-(D4-Pad2)
- R21 pad 2: Net-(D5-Pad5) -> Net-(D5-Pad2)
- R22 pad 2: Net-(D6-Pad5) -> Net-(D6-Pad2)
- R23 pad 2: Net-(D7-Pad5) -> Net-(D7-Pad2)
- R24 pad 2: Net-(D8-Pad5) -> Net-(D8-Pad2)
- R25 pad 2: Net-(D9-Pad5) -> Net-(D9-Pad2)
- R26 pad 2: Net-(D3-Pad4) -> Net-(D3-Pad1)
- R27 pad 2: Net-(D4-Pad4) -> Net-(D4-Pad1)
- R28 pad 2: Net-(D5-Pad4) -> Net-(D5-Pad1)
- R29 pad 2: Net-(D6-Pad4) -> Net-(D6-Pad1)
- R30 pad 2: Net-(D7-Pad4) -> Net-(D7-Pad1)
- R31 pad 2: Net-(D8-Pad4) -> Net-(D8-Pad1)
- R32 pad 2: Net-(D9-Pad4) -> Net-(D9-Pad1)
- R33 pad 2: Net-(D10-Pad6) -> Net-(D10-Pad3)
- R34 pad 2: Net-(D11-Pad6) -> Net-(D11-Pad3)
- R35 pad 2: Net-(D12-Pad6) -> Net-(D12-Pad3)
- R36 pad 2: Net-(D13-Pad6) -> Net-(D13-Pad3)
- R37 pad 2: Net-(D14-Pad6) -> Net-(D14-Pad3)
- R38 pad 2: Net-(D15-Pad6) -> Net-(D15-Pad3)
- R39 pad 2: Net-(D16-Pad6) -> Net-(D16-Pad3)
- R40 pad 2: Net-(D10-Pad5) -> Net-(D10-Pad2)
- R41 pad 2: Net-(D11-Pad5) -> Net-(D11-Pad2)
- R42 pad 2: Net-(D12-Pad5) -> Net-(D12-Pad2)
- R43 pad 2: Net-(D13-Pad5) -> Net-(D13-Pad2)
- R44 pad 2: Net-(D14-Pad5) -> Net-(D14-Pad2)
- R45 pad 2: Net-(D15-Pad5) -> Net-(D15-Pad2)
- R46 pad 2: Net-(D16-Pad5) -> Net-(D16-Pad2)
- R47 pad 2: Net-(D10-Pad4) -> Net-(D10-Pad1)
- R48 pad 2: Net-(D11-Pad4) -> Net-(D11-Pad1)
- R49 pad 2: Net-(D12-Pad4) -> Net-(D12-Pad1)
- R50 pad 2: Net-(D13-Pad4) -> Net-(D13-Pad1)
- R51 pad 2: Net-(D14-Pad4) -> Net-(D14-Pad1)
- R52 pad 2: Net-(D15-Pad4) -> Net-(D15-Pad1)
- R53 pad 2: Net-(D16-Pad4) -> Net-(D16-Pad1)
- R54 pad 2: Net-(D17-Pad6) -> Net-(D17-Pad3)
- R55 pad 2: Net-(D18-Pad6) -> Net-(D18-Pad3)
- R56 pad 2: Net-(D19-Pad6) -> Net-(D19-Pad3)
- R57 pad 2: Net-(D20-Pad6) -> Net-(D20-Pad3)
- R58 pad 2: Net-(D21-Pad6) -> Net-(D21-Pad3)
- R59 pad 2: Net-(D22-Pad6) -> Net-(D22-Pad3)
- R60 pad 2: Net-(D23-Pad6) -> Net-(D23-Pad3)
- R61 pad 2: Net-(D17-Pad5) -> Net-(D17-Pad2)
- R62 pad 2: Net-(D18-Pad5) -> Net-(D18-Pad2)
- R63 pad 2: Net-(D19-Pad5) -> Net-(D19-Pad2)
- R64 pad 2: Net-(D20-Pad5) -> Net-(D20-Pad2)
- R65 pad 2: Net-(D21-Pad5) -> Net-(D21-Pad2)
- R66 pad 2: Net-(D22-Pad5) -> Net-(D22-Pad2)
- R67 pad 2: Net-(D23-Pad5) -> Net-(D23-Pad2)
- R68 pad 2: Net-(D17-Pad4) -> Net-(D17-Pad1)
- R69 pad 2: Net-(D18-Pad4) -> Net-(D18-Pad1)
- R70 pad 2: Net-(D19-Pad4) -> Net-(D19-Pad1)
- R71 pad 2: Net-(D20-Pad4) -> Net-(D20-Pad1)
- R72 pad 2: Net-(D21-Pad4) -> Net-(D21-Pad1)
- R73 pad 2: Net-(D22-Pad4) -> Net-(D22-Pad1)
- R74 pad 2: Net-(D23-Pad4) -> Net-(D23-Pad1)
Routing:
- net GND: track 25.9 -> 104.4 mm, vias 26 -> 40
- net Net-(D7-Pad6): track 2.17 -> 0.00 mm
- net Net-(D7-Pad3): track 0.00 -> 2.17 mm
- net Net-(D4-Pad4): track 2.17 -> 0.00 mm
- net Net-(D4-Pad1): track 0.00 -> 2.17 mm
- net Net-(D11-Pad4): track 2.17 -> 0.00 mm
- net Net-(D11-Pad1): track 0.00 -> 2.17 mm
- net Net-(D10-Pad4): track 2.17 -> 0.00 mm
- net Net-(D10-Pad1): track 0.00 -> 2.17 mm
- net Net-(D19-Pad5): track 2.17 -> 0.00 mm
- net Net-(D19-Pad2): track 0.00 -> 2.17 mm
- net Net-(D16-Pad6): track 2.17 -> 0.00 mm
- net Net-(D16-Pad3): track 0.00 -> 2.17 mm
- net Net-(D15-Pad6): track 2.17 -> 0.00 mm
- net Net-(D15-Pad3): track 0.00 -> 2.17 mm
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
Commit message: Deleted LEDs' references
Other:
- board text added: "JLCJLCJLCJLC"
